Commit message: updated mesh file paths

File: obelisk_ws/src/robots/achilles_model/urdf/achilles.urdf (robot description, URDF)
Before this commit: robot achilles, 29 links, 28 joints
Links:
- link left_ankle_pitch: geometry visual mesh filename=package://achilles_model/meshes/ankle_pitch.STL
- link left_elbow_pitch: geometry visual mesh filename=package://achilles_model/meshes/left_elbow_pitch.STL
- link left_hip_pitch: geometry visual mesh filename=package://achilles_model/meshes/left_hip_pitch.STL
- link left_hip_roll: geometry visual mesh filename=package://achilles_model/meshes/left_hip_roll.STL
- link left_hip_yaw: geometry visual mesh filename=package://achilles_model/meshes/left_hip_yaw.STL
- link left_knee_pitch: geometry visual mesh filename=package://achilles_model/meshes/left_knee_pitch.STL
- link left_shoulder_pitch: geometry visual mesh filename=package://achilles_model/meshes/left_shoulder_pitch.STL
- link left_shoulder_roll: geometry visual mesh filename=package://achilles_model/meshes/left_shoulder_roll.STL
- link left_shoulder_yaw: geometry visual mesh filename=package://achilles_model/meshes/right_shoulder_yaw.STL
- link right_ankle_pitch: geometry visual mesh filename=package://achilles_model/meshes/ankle_pitch.STL
- link right_elbow_pitch: geometry visual mesh filename=package://achilles_model/meshes/right_elbow_pitch.STL
- link right_hip_pitch: geometry visual mesh filename=package://achilles_model/meshes/right_hip_pitch.STL
- link right_hip_roll: geometry visual mesh filename=package://achilles_model/meshes/right_hip_roll.STL
- link right_hip_yaw: geometry visual mesh filename=package://achilles_model/meshes/right_hip_yaw.STL
- link right_knee_pitch: geometry visual mesh filename=package://achilles_model/meshes/right_knee_pitch.STL
- link right_shoulder_pitch: geometry visual mesh filename=package://achilles_model/meshes/right_shoulder_pitch.STL
- link right_shoulder_roll: geometry visual mesh filename=package://achilles_model/meshes/right_shoulder_roll.STL
- link right_shoulder_yaw: geometry visual mesh filename=package://achilles_model/meshes/right_shoulder_yaw.STL
- link torso: geometry collision mesh filename=package://achilles_model/meshes/torso.STL; visual mesh filename=package://achilles_model/meshes/torso.STL
