Commit message: fix missing suffixes + make suffix optional

File: obelisk_ws/src/robots/leap_rh/urdf/leap_rh.urdf (robot description, URDF)
Before this commit: robot leap_rh, 17 links, 16 joints
Links:
- removed link if_bs_obk
- removed link if_ds_obk
- removed link if_md_obk
- removed link if_px_obk
- removed link mf_bs_obk
- removed link mf_ds_obk
- removed link mf_md_obk
- removed link mf_px_obk
- removed link palm_obk
- removed link rf_bs_obk
- removed link rf_ds_obk
- removed link rf_md_obk
- removed link rf_px_obk
- removed link th_bs_obk
- removed link th_ds_obk
- removed link th_mp_obk
- removed link th_px_obk
- added link if_bs, mass 0.044; collision box size=0.014 0.02 0.004; collision box size=0.014 0.02 0.004
- added link if_ds, mass 0.016; collision box size=0.014 0.022 0.004; collision box size=0.014 0.022 0.004
- added link if_md, mass 0.037; collision box size=0.014 0.02 0.004; collision box size=0.014 0.02 0.004
- added link if_px, mass 0.032; collision box size=0.034 0.026 0.022; visual mesh filename=package://leap_rh/meshes/proximal.obj
- added link mf_bs, mass 0.044; collision box size=0.014 0.02 0.004; collision box size=0.014 0.02 0.004
- added link mf_ds, mass 0.016; collision box size=0.014 0.022 0.004; collision box size=0.014 0.022 0.004
- added link mf_md, mass 0.037; collision box size=0.014 0.02 0.004; collision box size=0.014 0.02 0.004
- added link mf_px, mass 0.032; collision box size=0.034 0.026 0.022; visual mesh filename=package://leap_rh/meshes/proximal.obj
- added link palm, mass 0.237; collision box size=0.004 0.036 0.034; collision box size=0.01 0.12 0.02
- added link rf_bs, mass 0.044; collision box size=0.014 0.02 0.004; collision box size=0.014 0.02 0.004
- added link rf_ds, mass 0.016; collision box size=0.014 0.022 0.004; collision box size=0.014 0.022 0.004
- added link rf_md, mass 0.037; collision box size=0.014 0.02 0.004; collision box size=0.014 0.02 0.004
- added link rf_px, mass 0.032; collision box size=0.034 0.026 0.022; visual mesh filename=package://leap_rh/meshes/proximal.obj
- added link th_bs, mass 0.003; collision box size=0.014 0.004 0.02; collision box size=0.014 0.004 0.02
- added link th_ds, mass 0.049; collision box size=0.008 0.024 0.018; collision box size=0.02 0.004 0.03
- added link th_mp, mass 0.032; collision box size=0.034 0.026 0.022; visual mesh filename=package://leap_rh/meshes/proximal.obj
- added link th_px, mass 0.038; collision box size=0.01 0.024 0.018; collision box size=0.014 0.02 0.004
Joints:
- removed joint if_dip_obk
- removed joint if_mcp_obk
- removed joint if_pip_obk
- removed joint if_rot_obk
- removed joint mf_dip_obk
- removed joint mf_mcp_obk
- removed joint mf_pip_obk
- removed joint mf_rot_obk
- removed joint rf_dip_obk
- removed joint rf_mcp_obk
- removed joint rf_pip_obk
- removed joint rf_rot_obk
- removed joint th_axl_obk
- removed joint th_cmc_obk
- removed joint th_ipl_obk
- removed joint th_mcp_obk
- added joint if_dip: type revolute, parent if_md, child if_ds, origin xyz=0 -0.0361 0.0002 rpy=0 0 0, axis 0 0 -1, limit lower=-0.366 upper=2.042 effort=0.95 velocity=8.48
- added joint if_mcp: type revolute, parent palm, child if_bs, origin xyz=-0.0070 0.0230 -0.0187 rpy=1.57079 1.57079 0, axis 0 0 -1, limit lower=-0.314 upper=2.23 effort=0.95 velocity=8.48
- added joint if_pip: type revolute, parent if_px, child if_md, origin xyz=0.015 0.0143 -0.013 rpy=1.57079 -1.57079 0, axis 0 0 -1, limit lower=-0.506 upper=1.885 effort=0.95 velocity=8.48
- added joint if_rot: type revolute, parent if_bs, child if_px, origin xyz=-0.0122 0.03810 0.01450 rpy=-1.57079 0 1.57079, axis 0 0 -1, limit lower=-1.047 upper=1.047 effort=0.95 velocity=8.48
- added joint mf_dip: type revolute, parent mf_md, child mf_ds, origin xyz=0 -0.0361 0.0002 rpy=0 0 0, axis 0 0 -1, limit lower=-0.366 upper=2.042 effort=0.95 velocity=8.48
- added joint mf_mcp: type revolute, parent palm, child mf_bs, origin xyz=-0.0071 -0.0224 -0.0187 rpy=1.57079 1.57079 0, axis 0 0 -1, limit lower=-0.314 upper=2.23 effort=0.95 velocity=8.48
- added joint mf_pip: type revolute, parent mf_px, child mf_md, origin xyz=0.015 0.0143 -0.013 rpy=1.57079 -1.57079 0, axis 0 0 -1, limit lower=-0.506 upper=1.885 effort=0.95 velocity=8.48
- added joint mf_rot: type revolute, parent mf_bs, child mf_px, origin xyz=-0.0122 0.0381 0.0145 rpy=-1.57079 0 1.57079, axis 0 0 -1, limit lower=-1.047 upper=1.047 effort=0.95 velocity=8.48
- added joint rf_dip: type revolute, parent rf_md, child rf_ds, origin xyz=0 -0.03609 0.0002 rpy=0 0 0, axis 0 0 -1, limit lower=-0.366 upper=2.042 effort=0.95 velocity=8.48
- added joint rf_mcp: type revolute, parent palm, child rf_bs, origin xyz=-0.00709 -0.0678 -0.0187 rpy=1.57079 1.57079 0, axis 0 0 -1, limit lower=-0.314 upper=2.23 effort=0.95 velocity=8.48
- added joint rf_pip: type revolute, parent rf_px, child rf_md, origin xyz=0.015 0.0143 -0.013 rpy=1.57079 -1.57079 0, axis 0 0 -1, limit lower=-0.506 upper=1.885 effort=0.95 velocity=8.48
- added joint rf_rot: type revolute, parent rf_bs, child rf_px, origin xyz=-0.0122 0.0381 0.0145 rpy=-1.57079 0 1.57079, axis 0 0 -1, limit lower=-1.047 upper=1.047 effort=0.95 velocity=8.48
- added joint th_axl: type revolute, parent th_mp, child th_bs, origin xyz=0 0.0143 -0.013 rpy=1.57079 -1.57079 0, axis 0 0 -1, limit lower=-0.47 upper=2.443 effort=0.95 velocity=8.48
- added joint th_cmc: type revolute, parent palm, child th_mp, origin xyz=-0.0693 -0.0012 -0.0216 rpy=0 1.57079 0, axis 0 0 -1, limit lower=-0.349 upper=2.094 effort=0.95 velocity=8.48
- added joint th_ipl: type revolute, parent th_px, child th_ds, origin xyz=0 0.0466 0.0002 rpy=0 0 3.14159, axis 0 0 -1, limit lower=-1.34 upper=1.88 effort=0.95 velocity=8.48
- added joint th_mcp: type revolute, parent th_bs, child th_px, origin xyz=0 0.0145 -0.017 rpy=-1.57079 0 0, axis 0 0 -1, limit lower=-1.20 upper=1.90 effort=0.95 velocity=8.48

File: obelisk_ws/src/robots/leap_rh/urdf/leap_rh.urdf.xacro (robot description, xacro)
@@ -2,4 +2,4 @@
 <robot xmlns:xacro="http://ros.org/wiki/xacro" name="leap_rh">
   <xacro:include filename="leap_rh.xacro"/>
-  <xacro:leap_rh suffix="obk"/>
+  <xacro:leap_rh />
 </robot>

File: obelisk_ws/src/robots/leap_rh/urdf/leap_rh.xacro (robot description, xacro)
@@ -2,18 +2,19 @@
 <robot xmlns:xacro="http://ros.org/wiki/xacro" name="leap_rh">
   <!-- xacro -->
-  <xacro:macro name="leap_rh" params="collision:=True alpha:=1.0 suffix">
+  <xacro:macro name="leap_rh" params="collision:=True alpha:=1.0 suffix:=''">
+    <xacro:property name="optional_suffix" value="${'_' + suffix if suffix != '' else ''}" />
     <!-- palm -->
-    <link name="palm_${suffix}">
-      <visual name="palm_visual_${suffix}">
+    <link name="palm${optional_suffix}">
+      <visual name="palm_visual${optional_suffix}">
         <origin xyz="-0.0200 0.02575 -0.0347" rpy="0 0 0"/>
         <geometry>
           <mesh filename="package://leap_rh/meshes/palm.obj"/>
         </geometry>
-        <material name="black_${suffix}">
-          <color rgba="0.2 0.2 0.2 ${alpha}"/>
-        </material>
-      </visual>
-      <xacro:if value="${collision}">
-        <collision name="palm_collision_1_${suffix}">
+        <material name="black${optional_suffix}">
+          <color rgba="0.2 0.2 0.2 ${alpha}"/>
+        </material>
+      </visual>
+      <xacro:if value="${collision}">
+        <collision name="palm_collision_1${optional_suffix}">
           <origin xyz="-0.009 0.008 -0.011" rpy="0 0 0"/>
           <geometry>
@@ -21,5 +22,5 @@
           </geometry>
         </collision>
-        <collision name="palm_collision_2_${suffix}">
+        <collision name="palm_collision_2${optional_suffix}">
           <origin xyz="-0.009 -0.037 -0.011" rpy="0 0 0"/>
           <geometry>
@@ -27,5 +28,5 @@
           </geometry>
         </collision>
-        <collision name="palm_collision_3_${suffix}">
+        <collision name="palm_collision_3${optional_suffix}">
           <origin xyz="-0.009 -0.082 -0.011" rpy="0 0 0"/>
           <geometry>
@@ -33,5 +34,5 @@
           </geometry>
         </collision>
-        <collision name="palm_collision_4_${suffix}">
+        <collision name="palm_collision_4${optional_suffix}">
           <origin xyz="-0.066 -0.078 -0.0115" rpy="0 0 -0.2967"/>
           <geometry>
@@ -39,5 +40,5 @@
           </geometry>
         </collision>
-        <collision name="palm_collision_5_${suffix}">
+        <collision name="palm_collision_5${optional_suffix}">
           <origin xyz="-0.03 -0.035 -0.003" rpy="0 0 0"/>
           <geometry>
@@ -45,5 +46,5 @@
           </geometry>
         </collision>
-        <collision name="palm_collision_6_${suffix}">
+        <collision name="palm_collision_6${optional_suffix}">
           <origin xyz="-0.032 -0.035 -0.024" rpy="0 0.785 0"/>
           <geometry>
@@ -51,5 +52,5 @@
           </geometry>
         </collision>
-        <collision name="palm_collision_7_${suffix}">
+        <collision name="palm_collision_7${optional_suffix}">
           <origin xyz="-0.048 -0.033 -0.0115" rpy="0 0 0"/>
           <geometry>
@@ -57,5 +58,5 @@
           </geometry>
         </collision>
-        <collision name="palm_collision_8_${suffix}">
+        <collision name="palm_collision_8${optional_suffix}">
           <origin xyz="-0.078 -0.053 -0.0115" rpy="0 0 0"/>
           <geometry>
@@ -63,5 +64,5 @@
           </geometry>
         </collision>
-        <collision name="palm_collision_9_${suffix}">
+        <collision name="palm_collision_9${optional_suffix}">
           <origin xyz="-0.098 -0.009 -0.006" rpy="0 0 0"/>
           <geometry>
@@ -69,5 +70,5 @@
           </geometry>
         </collision>
-        <collision name="palm_collision_10_${suffix}">
+        <collision name="palm_collision_10${optional_suffix}">
           <origin xyz="-0.078 -0.003 0.01" rpy="0 0 0"/>
           <geometry>
@@ -83,24 +84,24 @@
     </link>
     <!-- index finger -->
-    <joint name="if_mcp_${suffix}" type="revolute">
+    <joint name="if_mcp${optional_suffix}" type="revolute">
       <origin xyz="-0.0070 0.0230 -0.0187" rpy="1.57079 1.57079 0"/>
-      <parent link="palm"/>
-      <child link="if_bs"/>
+      <parent link="palm${optional_suffix}"/>
+      <child link="if_bs${optional_suffix}"/>
       <axis xyz="0 0 -1"/>
       <limit effort="0.95" velocity="8.48" lower="-0.314" upper="2.23"/>
       <joint_properties friction="0.0"/>
     </joint>
-    <link name="if_bs_${suffix}">
-      <visual name="if_bs_visual_${suffix}">
+    <link name="if_bs${optional_suffix}">
+      <visual name="if_bs_visual${optional_suffix}">
         <origin xyz="0.0084 0.0077 0.01465" rpy="0 0 0"/>
         <geometry>
           <mesh filename="package://leap_rh/meshes/base.obj"/>
         </geometry>
-        <material name="black_${suffix}">
-          <color rgba="0.2 0.2 0.2 ${alpha}"/>
-        </material>
-      </visual>
-      <xacro:if value="${collision}">
-        <collision name="if_bs_collision_1_${suffix}">
+        <material name="black${optional_suffix}">
+          <color rgba="0.2 0.2 0.2 ${alpha}"/>
+        </material>
+      </visual>
+      <xacro:if value="${collision}">
+        <collision name="if_bs_collision_1${optional_suffix}">
           <origin xyz="0 0.018 0.0147" rpy="0 0 0"/>
           <geometry>
@@ -108,5 +109,5 @@
           </geometry>
         </collision>
-        <collision name="if_bs_collision_2_${suffix}">
+        <collision name="if_bs_collision_2${optional_suffix}">
           <origin xyz="-0.027 0.042 0.015" rpy="0 0 0"/>
           <geometry>
@@ -114,5 +115,5 @@
           </geometry>
         </collision>
-        <collision name="if_bs_collision_3_${suffix}">
+        <collision name="if_bs_collision_3${optional_suffix}">
           <origin xyz="-0.0262 0.02 0.0146" rpy="0 0 0"/>
           <geometry>
@@ -120,5 +121,5 @@
           </geometry>
         </collision>
-        <collision name="if_bs_collision_4_${suffix}">
+        <collision name="if_bs_collision_4${optional_suffix}">
           <origin xyz="-0.0295 0.035 0.029" rpy="0 0 0"/>
           <geometry>
@@ -126,5 +127,5 @@
           </geometry>
         </collision>
-        <collision name="if_bs_collision_5_${suffix}">
+        <collision name="if_bs_collision_5${optional_suffix}">
           <origin xyz="0 0.005 0.03" rpy="0 0 0"/>
           <geometry>
@@ -132,5 +133,5 @@
           </geometry>
         </collision>
-        <collision name="if_bs_collision_6_${suffix}">
+        <collision name="if_bs_collision_6${optional_suffix}">
           <origin xyz="0 0.005 -0.001" rpy="0 0 0"/>
           <geometry>
@@ -145,24 +146,24 @@
       </inertial>
     </link>
-    <joint name="if_rot_${suffix}" type="revolute">
+    <joint name="if_rot${optional_suffix}" type="revolute">
       <origin xyz="-0.0122 0.03810 0.01450" rpy="-1.57079 0 1.57079"/>
-      <parent link="if_bs"/>
-      <child link="if_px"/>
+      <parent link="if_bs${optional_suffix}"/>
+      <child link="if_px${optional_suffix}"/>
       <axis xyz="0 0 -1"/>
       <limit effort="0.95" velocity="8.48" lower="-1.047" upper="1.047"/>
       <joint_properties friction="0.0"/>
     </joint>
-    <link name="if_px_${suffix}">
-      <visual name="if_px_visual_${suffix}">
+    <link name="if_px${optional_suffix}">
+      <visual name="if_px_visual${optional_suffix}">
         <origin xyz="0.0096 0.0002 0.0007" rpy="-1.57079 -1.57079 0"/>
         <geometry>
           <mesh filename="package://leap_rh/meshes/proximal.obj"/>
         </geometry>
-        <material name="black_${suffix}">
-          <color rgba="0.2 0.2 0.2 ${alpha}"/>
-        </material>
-      </visual>
-      <xacro:if value="${collision}">
-        <collision name="if_px_collision_1_${suffix}">
+        <material name="black${optional_suffix}">
+          <color rgba="0.2 0.2 0.2 ${alpha}"/>
+        </material>
+      </visual>
+      <xacro:if value="${collision}">
+        <collision name="if_px_collision_1${optional_suffix}">
           <origin xyz="0.0075 -0.0002 -0.011" rpy="0 0 0"/>
           <geometry>
@@ -177,24 +178,24 @@
       </inertial>
     </link>
-    <joint name="if_pip_${suffix}" type="revolute">
+    <joint name="if_pip${optional_suffix}" type="revolute">
       <origin xyz="0.015 0.0143 -0.013" rpy="1.57079 -1.57079 0"/>
-      <parent link="if_px"/>
-      <child link="if_md"/>
+      <parent link="if_px${optional_suffix}"/>
+      <child link="if_md${optional_suffix}"/>
       <axis xyz="0 0 -1"/>
       <limit effort="0.95" velocity="8.48" lower="-0.506" upper="1.885"/>
       <joint_properties friction="0.0"/>
     </joint>
-    <link name="if_md_${suffix}">
-      <visual name="if_md_visual_${suffix}">
+    <link name="if_md${optional_suffix}">
+      <visual name="if_md_visual${optional_suffix}">
         <origin xyz="0.0211 -0.0084 0.0097" rpy="-3.1415926 0 0"/>
         <geometry>
           <mesh filename="package://leap_rh/meshes/medial.obj"/>
         </geometry>
-        <material name="black_${suffix}">
-          <color rgba="0.2 0.2 0.2 ${alpha}"/>
-        </material>
-      </visual>
-      <xacro:if value="${collision}">
-        <collision name="if_md_collision_1_${suffix}">
+        <material name="black${optional_suffix}">
+          <color rgba="0.2 0.2 0.2 ${alpha}"/>
+        </material>
+      </visual>
+      <xacro:if value="${collision}">
+        <collision name="if_md_collision_1${optional_suffix}">
           <origin xyz="0 -0.02 0.015" rpy="0 0 0"/>
           <geometry>
@@ -202,5 +203,5 @@
           </geometry>
         </collision>
-        <collision name="if_md_collision_2_${suffix}">
+        <collision name="if_md_collision_2${optional_suffix}">
           <origin xyz="0 -0.016 0.015" rpy="0 0 0"/>
           <geometry>
@@ -208,5 +209,5 @@
           </geometry>
         </collision>
-        <collision name="if_md_collision_3_${suffix}">
+        <collision name="if_md_collision_3${optional_suffix}">
           <origin xyz="0 -0.0045 0.03" rpy="0 0 0"/>
           <geometry>
@@ -214,5 +215,5 @@
           </geometry>
         </collision>
-        <collision name="if_md_collision_4_${suffix}">
+        <collision name="if_md_collision_4${optional_suffix}">
           <origin xyz="0 -0.0045 0" rpy="0 0 0"/>
           <geometry>
@@ -220,5 +221,5 @@
           </geometry>
         </collision>
-        <collision name="if_md_collision_5_${suffix}">
+        <collision name="if_md_collision_5${optional_suffix}">
           <origin xyz="0.0075 -0.035 0.015" rpy="0 0 0"/>
           <geometry>
@@ -233,24 +234,24 @@
       </inertial>
     </link>
-    <joint name="if_dip_${suffix}" type="revolute">
+    <joint name="if_dip${optional_suffix}" type="revolute">
       <origin xyz="0 -0.0361 0.0002" rpy="0 0 0"/>
-      <parent link="if_md"/>
-      <child link="if_ds"/>
+      <parent link="if_md${optional_suffix}"/>
+      <child link="if_ds${optional_suffix}"/>
       <axis xyz="0 0 -1"/>
       <limit effort="0.95" velocity="8.48" lower="-0.366" upper="2.042"/>
       <joint_properties friction="0.0"/>
     </joint>
-    <link name="if_ds_${suffix}">
-      <visual name="if_ds_visual_${suffix}">
+    <link name="if_ds${optional_suffix}">
+      <visual name="if_ds_visual${optional_suffix}">
         <origin xyz="0.0132 -0.0061 0.0144" rpy="3.1415926 0 0"/>
         <geometry>
           <mesh filename="package://leap_rh/meshes/distal.obj"/>
         </geometry>
-        <material name="black_${suffix}">
-          <color rgba="0.2 0.2 0.2 ${alpha}"/>
-        </material>
-      </visual>
-      <xacro:if value="${collision}">
-        <collision name="if_ds_collision_1_${suffix}">
+        <material name="black${optional_suffix}">
+          <color rgba="0.2 0.2 0.2 ${alpha}"/>
+        </material>
+      </visual>
+      <xacro:if value="${collision}">
+        <collision name="if_ds_collision_1${optional_suffix}">
           <origin xyz="0 -0.017 0.015" rpy="0 0 0"/>
           <geometry>
@@ -258,5 +259,5 @@
           </geometry>
         </collision>
-        <collision name="if_ds_collision_2_${suffix}">
+        <collision name="if_ds_collision_2${optional_suffix}">
           <origin xyz="0 -0.006 0.03" rpy="0 0 0"/>
           <geometry>
@@ -264,5 +265,5 @@
           </geometry>
         </collision>
-        <collision name="if_ds_collision_3_${suffix}">
+        <collision name="if_ds_collision_3${optional_suffix}">
           <origin xyz="0 -0.006 -0.001" rpy="0 0 0"/>
           <geometry>
@@ -270,5 +271,5 @@
           </geometry>
         </collision>
-        <collision name="if_ds_collision_4_${suffix}">
+        <collision name="if_ds_collision_4${optional_suffix}">
           <origin xyz="0 0 0" rpy="0 0 0"/>
           <geometry>
@@ -284,24 +285,24 @@
     </link>
     <!-- middle finger -->
-    <joint name="mf_mcp_${suffix}" type="revolute">
+    <joint name="mf_mcp${optional_suffix}" type="revolute">
       <origin xyz="-0.0071 -0.0224 -0.0187" rpy="1.57079 1.57079 0"/>
-      <parent link="palm"/>
-      <child link="mf_bs"/>
+      <parent link="palm${optional_suffix}"/>
+      <child link="mf_bs${optional_suffix}"/>
       <axis xyz="0 0 -1"/>
       <limit effort="0.95" velocity="8.48" lower="-0.314" upper="2.23"/>
       <joint_properties friction="0.0"/>
     </joint>
-    <link name="mf_bs_${suffix}">
-      <visual name="mf_bs_visual_${suffix}">
+    <link name="mf_bs${optional_suffix}">
+      <visual name="mf_bs_visual${optional_suffix}">
         <origin xyz="0.0084 0.0077 0.01465" rpy="0 0 0"/>
         <geometry>
           <mesh filename="package://leap_rh/meshes/base.obj"/>
         </geometry>
-        <material name="black_${suffix}">
-          <color rgba="0.2 0.2 0.2 ${alpha}"/>
-        </material>
-      </visual>
-      <xacro:if value="${collision}">
-        <collision name="mf_bs_collision_1_${suffix}">
+        <material name="black${optional_suffix}">
+          <color rgba="0.2 0.2 0.2 ${alpha}"/>
+        </material>
+      </visual>
+      <xacro:if value="${collision}">
+        <collision name="mf_bs_collision_1${optional_suffix}">
           <origin xyz="0 0.018 0.0147" rpy="0 0 0"/>
           <geometry>
@@ -309,5 +310,5 @@
           </geometry>
         </collision>
-        <collision name="mf_bs_collision_2_${suffix}">
+        <collision name="mf_bs_collision_2${optional_suffix}">
           <origin xyz="-0.027 0.042 0.015" rpy="0 0 0"/>
           <geometry>
@@ -315,5 +316,5 @@
           </geometry>
         </collision>
-        <collision name="mf_bs_collision_3_${suffix}">
+        <collision name="mf_bs_collision_3${optional_suffix}">
           <origin xyz="-0.0262 0.02 0.0146" rpy="0 0 0"/>
           <geometry>
@@ -321,5 +322,5 @@
           </geometry>
         </collision>
-        <collision name="mf_bs_collision_4_${suffix}">
+        <collision name="mf_bs_collision_4${optional_suffix}">
           <origin xyz="-0.0295 0.035 0.029" rpy="0 0 0"/>
           <geometry>
@@ -327,5 +328,5 @@
           </geometry>
         </collision>
-        <collision name="mf_bs_collision_5_${suffix}">
+        <collision name="mf_bs_collision_5${optional_suffix}">
           <origin xyz="0 0.005 0.03" rpy="0 0 0"/>
           <geometry>
@@ -333,5 +334,5 @@
           </geometry>
         </collision>
-        <collision name="mf_bs_collision_6_${suffix}">
+        <collision name="mf_bs_collision_6${optional_suffix}">
           <origin xyz="0 0.005 -0.001" rpy="0 0 0"/>
           <geometry>
@@ -346,24 +347,24 @@
       </inertial>
     </link>
-    <joint name="mf_rot_${suffix}" type="revolute">
+    <joint name="mf_rot${optional_suffix}" type="revolute">
       <origin xyz="-0.0122 0.0381 0.0145" rpy="-1.57079 0 1.57079"/>
-      <parent link="mf_bs"/>
-      <child link="mf_px"/>
+      <parent link="mf_bs${optional_suffix}"/>
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