Commit message: allow leap hand to be configurable with alpha and conditional collision geoms

File: obelisk_ws/src/robots/leap_rh/urdf/leap_rh.xacro (robot description, xacro)
@@ -2,5 +2,5 @@
 <robot xmlns:xacro="http://ros.org/wiki/xacro" name="leap_rh">
   <!-- xacro -->
-  <xacro:macro name="leap_rh">
+  <xacro:macro name="leap_rh" params="collision:=true alpha:=1.0">
     <!-- palm -->
     <link name="palm">
@@ -11,67 +11,69 @@
         </geometry>
         <material name="black">
-          <color rgba="0.2 0.2 0.2 1"/>
-        </material>
-      </visual>
-      <collision name="palm_collision_1">
-        <origin xyz="-0.009 0.008 -0.011" rpy="0 0 0"/>
-        <geometry>
-          <box size="0.022 0.026 0.034"/>
-        </geometry>
-      </collision>
-      <collision name="palm_collision_2">
-        <origin xyz="-0.009 -0.037 -0.011" rpy="0 0 0"/>
-        <geometry>
-          <box size="0.022 0.026 0.034"/>
-        </geometry>
-      </collision>
-      <collision name="palm_collision_3">
-        <origin xyz="-0.009 -0.082 -0.011" rpy="0 0 0"/>
-        <geometry>
-          <box size="0.022 0.026 0.034"/>
-        </geometry>
-      </collision>
-      <collision name="palm_collision_4">
-        <origin xyz="-0.066 -0.078 -0.0115" rpy="0 0 -0.2967"/>
-        <geometry>
-          <box size="0.058 0.02 0.046"/>
-        </geometry>
-      </collision>
-      <collision name="palm_collision_5">
-        <origin xyz="-0.03 -0.035 -0.003" rpy="0 0 0"/>
-        <geometry>
-          <box size="0.02 0.12 0.03"/>
-        </geometry>
-      </collision>
-      <collision name="palm_collision_6">
-        <origin xyz="-0.032 -0.035 -0.024" rpy="0 0.785 0"/>
-        <geometry>
-          <box size="0.01 0.12 0.02"/>
-        </geometry>
-      </collision>
-      <collision name="palm_collision_7">
-        <origin xyz="-0.048 -0.033 -0.0115" rpy="0 0 0"/>
-        <geometry>
-          <box size="0.024 0.116 0.046"/>
-        </geometry>
-      </collision>
-      <collision name="palm_collision_8">
-        <origin xyz="-0.078 -0.053 -0.0115" rpy="0 0 0"/>
-        <geometry>
-          <box size="0.044 0.052 0.046"/>
-        </geometry>
-      </collision>
-      <collision name="palm_collision_9">
-        <origin xyz="-0.098 -0.009 -0.006" rpy="0 0 0"/>
-        <geometry>
-          <box size="0.004 0.036 0.034"/>
-        </geometry>
-      </collision>
-      <collision name="palm_collision_10">
-        <origin xyz="-0.078 -0.003 0.01" rpy="0 0 0"/>
-        <geometry>
-          <box size="0.044 0.056 0.004"/>
-        </geometry>
-      </collision>
+          <color rgba="0.2 0.2 0.2 ${alpha}"/>
+        </material>
+      </visual>
+      <xacro:if value="${collision == 'true'}">
+        <collision name="palm_collision_1">
+          <origin xyz="-0.009 0.008 -0.011" rpy="0 0 0"/>
+          <geometry>
+            <box size="0.022 0.026 0.034"/>
+          </geometry>
+        </collision>
+        <collision name="palm_collision_2">
+          <origin xyz="-0.009 -0.037 -0.011" rpy="0 0 0"/>
+          <geometry>
+            <box size="0.022 0.026 0.034"/>
+          </geometry>
+        </collision>
+        <collision name="palm_collision_3">
+          <origin xyz="-0.009 -0.082 -0.011" rpy="0 0 0"/>
+          <geometry>
+            <box size="0.022 0.026 0.034"/>
+          </geometry>
+        </collision>
+        <collision name="palm_collision_4">
+          <origin xyz="-0.066 -0.078 -0.0115" rpy="0 0 -0.2967"/>
+          <geometry>
+            <box size="0.058 0.02 0.046"/>
+          </geometry>
+        </collision>
+        <collision name="palm_collision_5">
+          <origin xyz="-0.03 -0.035 -0.003" rpy="0 0 0"/>
+          <geometry>
+            <box size="0.02 0.12 0.03"/>
+          </geometry>
+        </collision>
+        <collision name="palm_collision_6">
+          <origin xyz="-0.032 -0.035 -0.024" rpy="0 0.785 0"/>
+          <geometry>
+            <box size="0.01 0.12 0.02"/>
+          </geometry>
+        </collision>
+        <collision name="palm_collision_7">
+          <origin xyz="-0.048 -0.033 -0.0115" rpy="0 0 0"/>
+          <geometry>
+            <box size="0.024 0.116 0.046"/>
+          </geometry>
+        </collision>
+        <collision name="palm_collision_8">
+          <origin xyz="-0.078 -0.053 -0.0115" rpy="0 0 0"/>
+          <geometry>
+            <box size="0.044 0.052 0.046"/>
+          </geometry>
+        </collision>
+        <collision name="palm_collision_9">
+          <origin xyz="-0.098 -0.009 -0.006" rpy="0 0 0"/>
+          <geometry>
+            <box size="0.004 0.036 0.034"/>
+          </geometry>
+        </collision>
+        <collision name="palm_collision_10">
+          <origin xyz="-0.078 -0.003 0.01" rpy="0 0 0"/>
+          <geometry>
+            <box size="0.044 0.056 0.004"/>
+          </geometry>
+        </collision>
+      </xacro:if>
       <inertial>
         <origin rpy="0 0 0" xyz="-0.049542 -0.042914 -0.010227"/>
@@ -96,43 +98,45 @@
         </geometry>
         <material name="black">
-          <color rgba="0.2 0.2 0.2 1"/>
-        </material>
-      </visual>
-      <collision name="if_bs_collision_1">
-        <origin xyz="0 0.018 0.0147" rpy="0 0 0"/>
-        <geometry>
-          <box size="0.02 0.006 0.034"/>
-        </geometry>
-      </collision>
-      <collision name="if_bs_collision_2">
-        <origin xyz="-0.027 0.042 0.015" rpy="0 0 0"/>
-        <geometry>
-          <box size="0.028 0.04 0.02"/>
-        </geometry>
-      </collision>
-      <collision name="if_bs_collision_3">
-        <origin xyz="-0.0262 0.02 0.0146" rpy="0 0 0"/>
-        <geometry>
-          <box size="0.034 0.006 0.02"/>
-        </geometry>
-      </collision>
-      <collision name="if_bs_collision_4">
-        <origin xyz="-0.0295 0.035 0.029" rpy="0 0 0"/>
-        <geometry>
-          <box size="0.02 0.024 0.008"/>
-        </geometry>
-      </collision>
-      <collision name="if_bs_collision_5">
-        <origin xyz="0 0.005 0.03" rpy="0 0 0"/>
-        <geometry>
-          <box size="0.014 0.02 0.004"/>
-        </geometry>
-      </collision>
-      <collision name="if_bs_collision_6">
-        <origin xyz="0 0.005 -0.001" rpy="0 0 0"/>
-        <geometry>
-          <box size="0.014 0.02 0.004"/>
-        </geometry>
-      </collision>
+          <color rgba="0.2 0.2 0.2 ${alpha}"/>
+        </material>
+      </visual>
+      <xacro:if value="${collision == 'true'}">
+        <collision name="if_bs_collision_1">
+          <origin xyz="0 0.018 0.0147" rpy="0 0 0"/>
+          <geometry>
+            <box size="0.02 0.006 0.034"/>
+          </geometry>
+        </collision>
+        <collision name="if_bs_collision_2">
+          <origin xyz="-0.027 0.042 0.015" rpy="0 0 0"/>
+          <geometry>
+            <box size="0.028 0.04 0.02"/>
+          </geometry>
+        </collision>
+        <collision name="if_bs_collision_3">
+          <origin xyz="-0.0262 0.02 0.0146" rpy="0 0 0"/>
+          <geometry>
+            <box size="0.034 0.006 0.02"/>
+          </geometry>
+        </collision>
+        <collision name="if_bs_collision_4">
+          <origin xyz="-0.0295 0.035 0.029" rpy="0 0 0"/>
+          <geometry>
+            <box size="0.02 0.024 0.008"/>
+          </geometry>
+        </collision>
+        <collision name="if_bs_collision_5">
+          <origin xyz="0 0.005 0.03" rpy="0 0 0"/>
+          <geometry>
+            <box size="0.014 0.02 0.004"/>
+          </geometry>
+        </collision>
+        <collision name="if_bs_collision_6">
+          <origin xyz="0 0.005 -0.001" rpy="0 0 0"/>
+          <geometry>
+            <box size="0.014 0.02 0.004"/>
+          </geometry>
+        </collision>
+      </xacro:if>
       <inertial>
         <origin rpy="0 0 0" xyz="-0.022516 0.033882 0.016359"/>
@@ -156,13 +160,15 @@
         </geometry>
         <material name="black">
-          <color rgba="0.2 0.2 0.2 1"/>
-        </material>
-      </visual>
-      <collision name="if_px_collision_1">
-        <origin xyz="0.0075 -0.0002 -0.011" rpy="0 0 0"/>
-        <geometry>
-          <box size="0.034 0.026 0.022"/>
-        </geometry>
-      </collision>
+          <color rgba="0.2 0.2 0.2 ${alpha}"/>
+        </material>
+      </visual>
+      <xacro:if value="${collision == 'true'}">
+        <collision name="if_px_collision_1">
+          <origin xyz="0.0075 -0.0002 -0.011" rpy="0 0 0"/>
+          <geometry>
+            <box size="0.034 0.026 0.022"/>
+          </geometry>
+        </collision>
+      </xacro:if>
       <inertial>
         <origin rpy="0 0 0" xyz="0.0075 -0.0002 -0.011"/>
@@ -186,37 +192,39 @@
         </geometry>
         <material name="black">
-          <color rgba="0.2 0.2 0.2 1"/>
-        </material>
-      </visual>
-      <collision name="if_md_collision_1">
-        <origin xyz="0 -0.02 0.015" rpy="0 0 0"/>
-        <geometry>
-          <box size="0.016 0.006 0.026"/>
-        </geometry>
-      </collision>
-      <collision name="if_md_collision_2">
-        <origin xyz="0 -0.016 0.015" rpy="0 0 0"/>
-        <geometry>
-          <box size="0.02 0.004 0.034"/>
-        </geometry>
-      </collision>
-      <collision name="if_md_collision_3">
-        <origin xyz="0 -0.0045 0.03" rpy="0 0 0"/>
-        <geometry>
-          <box size="0.014 0.02 0.004"/>
-        </geometry>
-      </collision>
-      <collision name="if_md_collision_4">
-        <origin xyz="0 -0.0045 0" rpy="0 0 0"/>
-        <geometry>
-          <box size="0.014 0.02 0.004"/>
-        </geometry>
-      </collision>
-      <collision name="if_md_collision_5">
-        <origin xyz="0.0075 -0.035 0.015" rpy="0 0 0"/>
-        <geometry>
-          <box size="0.034 0.022 0.026"/>
-        </geometry>
-      </collision>
+          <color rgba="0.2 0.2 0.2 ${alpha}"/>
+        </material>
+      </visual>
+      <xacro:if value="${collision == 'true'}">
+        <collision name="if_md_collision_1">
+          <origin xyz="0 -0.02 0.015" rpy="0 0 0"/>
+          <geometry>
+            <box size="0.016 0.006 0.026"/>
+          </geometry>
+        </collision>
+        <collision name="if_md_collision_2">
+          <origin xyz="0 -0.016 0.015" rpy="0 0 0"/>
+          <geometry>
+            <box size="0.02 0.004 0.034"/>
+          </geometry>
+        </collision>
+        <collision name="if_md_collision_3">
+          <origin xyz="0 -0.0045 0.03" rpy="0 0 0"/>
+          <geometry>
+            <box size="0.014 0.02 0.004"/>
+          </geometry>
+        </collision>
+        <collision name="if_md_collision_4">
+          <origin xyz="0 -0.0045 0" rpy="0 0 0"/>
+          <geometry>
+            <box size="0.014 0.02 0.004"/>
+          </geometry>
+        </collision>
+        <collision name="if_md_collision_5">
+          <origin xyz="0.0075 -0.035 0.015" rpy="0 0 0"/>
+          <geometry>
+            <box size="0.034 0.022 0.026"/>
+          </geometry>
+        </collision>
+      </xacro:if>
       <inertial>
         <origin rpy="0 0 0" xyz="0.0054215 -0.029148 0.015"/>
@@ -240,31 +248,33 @@
         </geometry>
         <material name="black">
-          <color rgba="0.2 0.2 0.2 1"/>
-        </material>
-      </visual>
-      <collision name="if_ds_collision_1">
-        <origin xyz="0 -0.017 0.015" rpy="0 0 0"/>
-        <geometry>
-          <box size="0.02 0.006 0.03"/>
-        </geometry>
-      </collision>
-      <collision name="if_ds_collision_2">
-        <origin xyz="0 -0.006 0.03" rpy="0 0 0"/>
-        <geometry>
-          <box size="0.014 0.022 0.004"/>
-        </geometry>
-      </collision>
-      <collision name="if_ds_collision_3">
-        <origin xyz="0 -0.006 -0.001" rpy="0 0 0"/>
-        <geometry>
-          <box size="0.014 0.022 0.004"/>
-        </geometry>
-      </collision>
-      <collision name="if_ds_collision_4">
-        <origin xyz="0 0 0" rpy="0 0 0"/>
-        <geometry>
-          <mesh filename="package://leap_rh/meshes/tip.obj"/>
-        </geometry>
-      </collision>
+          <color rgba="0.2 0.2 0.2 ${alpha}"/>
+        </material>
+      </visual>
+      <xacro:if value="${collision == 'true'}">
+        <collision name="if_ds_collision_1">
+          <origin xyz="0 -0.017 0.015" rpy="0 0 0"/>
+          <geometry>
+            <box size="0.02 0.006 0.03"/>
+          </geometry>
+        </collision>
+        <collision name="if_ds_collision_2">
+          <origin xyz="0 -0.006 0.03" rpy="0 0 0"/>
+          <geometry>
+            <box size="0.014 0.022 0.004"/>
+          </geometry>
+        </collision>
+        <collision name="if_ds_collision_3">
+          <origin xyz="0 -0.006 -0.001" rpy="0 0 0"/>
+          <geometry>
+            <box size="0.014 0.022 0.004"/>
+          </geometry>
+        </collision>
+        <collision name="if_ds_collision_4">
+          <origin xyz="0 0 0" rpy="0 0 0"/>
+          <geometry>
+            <mesh filename="package://leap_rh/meshes/tip.obj"/>
+          </geometry>
+        </collision>
+      </xacro:if>
       <inertial>
         <origin rpy="0 0 0" xyz="-0.0008794 -0.027019 0.014594"/>
@@ -289,43 +299,45 @@
         </geometry>
         <material name="black">
-          <color rgba="0.2 0.2 0.2 1"/>
-        </material>
-      </visual>
-      <collision name="mf_bs_collision_1">
-        <origin xyz="0 0.018 0.0147" rpy="0 0 0"/>
-        <geometry>
-          <box size="0.02 0.006 0.034"/>
-        </geometry>
-      </collision>
-      <collision name="mf_bs_collision_2">
-        <origin xyz="-0.027 0.042 0.015" rpy="0 0 0"/>
-        <geometry>
-          <box size="0.028 0.04 0.02"/>
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
Commit message: remove suffixes from joint names and material names

File: obelisk_ws/src/robots/leap_rh/urdf/leap_rh.xacro (robot description, xacro)
@@ -11,5 +11,5 @@
           <mesh filename="package://leap_rh/meshes/palm.obj"/>
         </geometry>
-        <material name="black${optional_suffix}">
+        <material name="black">
           <color rgba="0.2 0.2 0.2 ${alpha}"/>
         </material>
@@ -84,5 +84,5 @@
     </link>
     <!-- index finger -->
-    <joint name="if_mcp${optional_suffix}" type="revolute">
+    <joint name="if_mcp" type="revolute">
       <origin xyz="-0.0070 0.0230 -0.0187" rpy="1.57079 1.57079 0"/>
       <parent link="palm${optional_suffix}"/>
@@ -98,5 +98,5 @@
           <mesh filename="package://leap_rh/meshes/base.obj"/>
         </geometry>
-        <material name="black${optional_suffix}">
+        <material name="black">
           <color rgba="0.2 0.2 0.2 ${alpha}"/>
         </material>
@@ -146,5 +146,5 @@
       </inertial>
     </link>
-    <joint name="if_rot${optional_suffix}" type="revolute">
+    <joint name="if_rot" type="revolute">
       <origin xyz="-0.0122 0.03810 0.01450" rpy="-1.57079 0 1.57079"/>
       <parent link="if_bs${optional_suffix}"/>
@@ -160,5 +160,5 @@
           <mesh filename="package://leap_rh/meshes/proximal.obj"/>
         </geometry>
-        <material name="black${optional_suffix}">
+        <material name="black">
           <color rgba="0.2 0.2 0.2 ${alpha}"/>
         </material>
@@ -178,5 +178,5 @@
       </inertial>
     </link>
-    <joint name="if_pip${optional_suffix}" type="revolute">
+    <joint name="if_pip" type="revolute">
       <origin xyz="0.015 0.0143 -0.013" rpy="1.57079 -1.57079 0"/>
       <parent link="if_px${optional_suffix}"/>
@@ -192,5 +192,5 @@
           <mesh filename="package://leap_rh/meshes/medial.obj"/>
         </geometry>
-        <material name="black${optional_suffix}">
+        <material name="black">
           <color rgba="0.2 0.2 0.2 ${alpha}"/>
         </material>
@@ -234,5 +234,5 @@
       </inertial>
     </link>
-    <joint name="if_dip${optional_suffix}" type="revolute">
+    <joint name="if_dip" type="revolute">
       <origin xyz="0 -0.0361 0.0002" rpy="0 0 0"/>
       <parent link="if_md${optional_suffix}"/>
@@ -248,5 +248,5 @@
           <mesh filename="package://leap_rh/meshes/distal.obj"/>
         </geometry>
-        <material name="black${optional_suffix}">
+        <material name="black">
           <color rgba="0.2 0.2 0.2 ${alpha}"/>
         </material>
@@ -285,5 +285,5 @@
     </link>
     <!-- middle finger -->
-    <joint name="mf_mcp${optional_suffix}" type="revolute">
+    <joint name="mf_mcp" type="revolute">
       <origin xyz="-0.0071 -0.0224 -0.0187" rpy="1.57079 1.57079 0"/>
       <parent link="palm${optional_suffix}"/>
@@ -299,5 +299,5 @@
           <mesh filename="package://leap_rh/meshes/base.obj"/>
         </geometry>
-        <material name="black${optional_suffix}">
+        <material name="black">
           <color rgba="0.2 0.2 0.2 ${alpha}"/>
         </material>
@@ -347,5 +347,5 @@
       </inertial>
     </link>
-    <joint name="mf_rot${optional_suffix}" type="revolute">
+    <joint name="mf_rot" type="revolute">
       <origin xyz="-0.0122 0.0381 0.0145" rpy="-1.57079 0 1.57079"/>
       <parent link="mf_bs${optional_suffix}"/>
@@ -361,5 +361,5 @@
           <mesh filename="package://leap_rh/meshes/proximal.obj"/>
         </geometry>
-        <material name="black${optional_suffix}">
+        <material name="black">
           <color rgba="0.2 0.2 0.2 ${alpha}"/>
         </material>
@@ -379,5 +379,5 @@
       </inertial>
     </link>
-    <joint name="mf_pip${optional_suffix}" type="revolute">
+    <joint name="mf_pip" type="revolute">
       <origin xyz="0.015 0.0143 -0.013" rpy="1.57079 -1.57079 0"/>
       <parent link="mf_px${optional_suffix}"/>
@@ -393,5 +393,5 @@
           <mesh filename="package://leap_rh/meshes/medial.obj"/>
         </geometry>
-        <material name="black${optional_suffix}">
+        <material name="black">
           <color rgba="0.2 0.2 0.2 ${alpha}"/>
         </material>
@@ -435,5 +435,5 @@
       </inertial>
     </link>
-    <joint name="mf_dip${optional_suffix}" type="revolute">
+    <joint name="mf_dip" type="revolute">
       <origin xyz="0 -0.0361 0.0002" rpy="0 0 0"/>
       <parent link="mf_md${optional_suffix}"/>
@@ -449,5 +449,5 @@
           <mesh filename="package://leap_rh/meshes/distal.obj"/>
         </geometry>
-        <material name="black${optional_suffix}">
+        <material name="black">
           <color rgba="0.2 0.2 0.2 ${alpha}"/>
         </material>
@@ -486,5 +486,5 @@
     </link>
     <!-- ring finger -->
-    <joint name="rf_mcp${optional_suffix}" type="revolute">
+    <joint name="rf_mcp" type="revolute">
       <origin xyz="-0.00709 -0.0678 -0.0187" rpy="1.57079 1.57079 0"/>
       <parent link="palm${optional_suffix}"/>
@@ -500,5 +500,5 @@
           <mesh filename="package://leap_rh/meshes/base.obj"/>
         </geometry>
-        <material name="black${optional_suffix}">
+        <material name="black">
           <color rgba="0.2 0.2 0.2 ${alpha}"/>
         </material>
@@ -548,5 +548,5 @@
       </inertial>
     </link>
-    <joint name="rf_rot${optional_suffix}" type="revolute">
+    <joint name="rf_rot" type="revolute">
       <origin xyz="-0.0122 0.0381 0.0145" rpy="-1.57079 0 1.57079"/>
       <parent link="rf_bs${optional_suffix}"/>
@@ -562,5 +562,5 @@
           <mesh filename="package://leap_rh/meshes/proximal.obj"/>
         </geometry>
-        <material name="black${optional_suffix}">
+        <material name="black">
           <color rgba="0.2 0.2 0.2 ${alpha}"/>
         </material>
@@ -580,5 +580,5 @@
       </inertial>
     </link>
-    <joint name="rf_pip${optional_suffix}" type="revolute">
+    <joint name="rf_pip" type="revolute">
       <origin xyz="0.015 0.0143 -0.013" rpy="1.57079 -1.57079 0"/>
       <parent link="rf_px${optional_suffix}"/>
@@ -594,5 +594,5 @@
           <mesh filename="package://leap_rh/meshes/medial.obj"/>
         </geometry>
-        <material name="black${optional_suffix}">
+        <material name="black">
           <color rgba="0.2 0.2 0.2 ${alpha}"/>
         </material>
@@ -636,5 +636,5 @@
       </inertial>
     </link>
-    <joint name="rf_dip${optional_suffix}" type="revolute">
+    <joint name="rf_dip" type="revolute">
       <origin xyz="0 -0.03609 0.0002" rpy="0 0 0"/>
       <parent link="rf_md${optional_suffix}"/>
@@ -650,5 +650,5 @@
           <mesh filename="package://leap_rh/meshes/distal.obj"/>
         </geometry>
-        <material name="black${optional_suffix}">
+        <material name="black">
           <color rgba="0.2 0.2 0.2 ${alpha}"/>
         </material>
@@ -687,5 +687,5 @@
     </link>
     <!-- thumb -->
-    <joint name="th_cmc${optional_suffix}" type="revolute">
+    <joint name="th_cmc" type="revolute">
       <origin xyz="-0.0693 -0.0012 -0.0216" rpy="0 1.57079 0"/>
       <parent link="palm${optional_suffix}"/>
@@ -701,5 +701,5 @@
           <mesh filename="package://leap_rh/meshes/proximal.obj"/>
         </geometry>
-        <material name="black${optional_suffix}">
+        <material name="black">
           <color rgba="0.2 0.2 0.2 ${alpha}"/>
         </material>
@@ -719,5 +719,5 @@
       </inertial>
     </link>
-    <joint name="th_axl${optional_suffix}" type="revolute">
+    <joint name="th_axl" type="revolute">
       <origin xyz="0 0.0143 -0.013" rpy="1.57079 -1.57079 0"/>
       <parent link="th_mp${optional_suffix}"/>
@@ -733,5 +733,5 @@
           <mesh filename="package://leap_rh/meshes/thumb_base.obj"/>
         </geometry>
-        <material name="black${optional_suffix}">
+        <material name="black">
           <color rgba="0.2 0.2 0.2 ${alpha}"/>
         </material>
@@ -763,5 +763,5 @@
       </inertial>
     </link>
-    <joint name="th_mcp${optional_suffix}" type="revolute">
+    <joint name="th_mcp" type="revolute">
       <origin xyz="0 0.0145 -0.017" rpy="-1.57079 0 0"/>
       <parent link="th_bs${optional_suffix}"/>
@@ -777,5 +777,5 @@
           <mesh filename="package://leap_rh/meshes/thumb_proximal.obj"/>
         </geometry>
-        <material name="black${optional_suffix}">
+        <material name="black">
           <color rgba="0.2 0.2 0.2 ${alpha}"/>
         </material>
@@ -819,5 +819,5 @@
       </inertial>
     </link>
-    <joint name="th_ipl${optional_suffix}" type="revolute">
+    <joint name="th_ipl" type="revolute">
       <origin xyz="0 0.0466 0.0002" rpy="0 0 3.14159"/>
       <parent link="th_px${optional_suffix}"/>
@@ -833,5 +833,5 @@
           <mesh filename="package://leap_rh/meshes/thumb_distal.obj"/>
         </geometry>
-        <material name="black${optional_suffix}">
+        <material name="black">
           <color rgba="0.2 0.2 0.2 ${alpha}"/>
         </material>
