Commit message: reading IMU and joint data from the robot. visualized and verified the data

File: obelisk_ws/src/robots/g1_description/urdf/g1.urdf (robot description, URDF)
Before this commit: robot g1, 44 links, 43 joints
Links:
- removed link left_elbow_pitch_link
- removed link left_elbow_roll_link
- removed link left_five_link
- removed link left_four_link
- removed link left_one_link
- removed link left_palm_link
- removed link left_six_link
- removed link left_three_link
- removed link left_two_link
- removed link left_zero_link
- removed link right_elbow_pitch_link
- removed link right_elbow_roll_link
- removed link right_five_link
- removed link right_four_link
- removed link right_one_link
- removed link right_palm_link
- removed link right_six_link
- removed link right_three_link
- removed link right_two_link
- removed link right_zero_link
- added link d435_link
- added link left_elbow_link, mass 0.6; collision mesh filename=package://g1_description/meshes/left_elbow_link.STL; visual mesh filename=package://g1_description/meshes/left_elbow_link.STL
- added link left_hand_index_0_link, mass 0.05885070; collision mesh filename=package://g1_description/meshes/left_hand_index_0_link.STL; visual mesh filename=package://g1_description/meshes/left_hand_index_0_link.STL
- added link left_hand_index_1_link, mass 0.02030626; collision mesh filename=package://g1_description/meshes/left_hand_index_1_link.STL; visual mesh filename=package://g1_description/meshes/left_hand_index_1_link.STL
- added link left_hand_middle_0_link, mass 0.05885070; collision mesh filename=package://g1_description/meshes/left_hand_middle_0_link.STL; visual mesh filename=package://g1_description/meshes/left_hand_middle_0_link.STL
- added link left_hand_middle_1_link, mass 0.02030626; collision mesh filename=package://g1_description/meshes/left_hand_middle_1_link.STL; visual mesh filename=package://g1_description/meshes/left_hand_middle_1_link.STL
- added link left_hand_palm_link, mass 0.37283854; collision mesh filename=package://g1_description/meshes/left_hand_palm_link.STL; visual mesh filename=package://g1_description/meshes/left_hand_palm_link.STL
- added link left_hand_thumb_0_link, mass 0.08623657; collision mesh filename=package://g1_description/meshes/left_hand_thumb_0_link.STL; visual mesh filename=package://g1_description/meshes/left_hand_thumb_0_link.STL
- added link left_hand_thumb_1_link, mass 0.05885070; collision box size=0.02 0.03 0.02; visual mesh filename=package://g1_description/meshes/left_hand_thumb_1_link.STL
- added link left_hand_thumb_2_link, mass 0.02030626; collision mesh filename=package://g1_description/meshes/left_hand_thumb_2_link.STL; visual mesh filename=package://g1_description/meshes/left_hand_thumb_2_link.STL
- added link left_heel
- added link left_toe
- added link left_wrist_pitch_link, mass 0.48404956; collision mesh filename=package://g1_description/meshes/left_wrist_pitch_link.STL; visual mesh filename=package://g1_description/meshes/left_wrist_pitch_link.STL
- added link left_wrist_roll_link, mass 0.08544498; collision mesh filename=package://g1_description/meshes/left_wrist_roll_link.STL; visual mesh filename=package://g1_description/meshes/left_wrist_roll_link.STL
- added link left_wrist_yaw_link, mass 0.08457647; collision mesh filename=package://g1_description/meshes/left_wrist_yaw_link.STL; visual mesh filename=package://g1_description/meshes/left_wrist_yaw_link.STL
- added link mid360_link
- added link right_elbow_link, mass 0.6; collision mesh filename=package://g1_description/meshes/right_elbow_link.STL; visual mesh filename=package://g1_description/meshes/right_elbow_link.STL
- added link right_hand_index_0_link, mass 0.05885070; collision mesh filename=package://g1_description/meshes/right_hand_index_0_link.STL; visual mesh filename=package://g1_description/meshes/right_hand_index_0_link.STL
- added link right_hand_index_1_link, mass 0.02030626; collision mesh filename=package://g1_description/meshes/right_hand_index_1_link.STL; visual mesh filename=package://g1_description/meshes/right_hand_index_1_link.STL
- added link right_hand_middle_0_link, mass 0.05885070; collision mesh filename=package://g1_description/meshes/right_hand_middle_0_link.STL; visual mesh filename=package://g1_description/meshes/right_hand_middle_0_link.STL
- added link right_hand_middle_1_link, mass 0.02030626; collision mesh filename=package://g1_description/meshes/right_hand_middle_1_link.STL; visual mesh filename=package://g1_description/meshes/right_hand_middle_1_link.STL
- added link right_hand_palm_link, mass 0.37283854; collision mesh filename=package://g1_description/meshes/right_hand_palm_link.STL; visual mesh filename=package://g1_description/meshes/right_hand_palm_link.STL
- added link right_hand_thumb_0_link, mass 0.08623657; collision mesh filename=package://g1_description/meshes/right_hand_thumb_0_link.STL; visual mesh filename=package://g1_description/meshes/right_hand_thumb_0_link.STL
- added link right_hand_thumb_1_link, mass 0.05885070; collision box size=0.02 0.03 0.02; visual mesh filename=package://g1_description/meshes/right_hand_thumb_1_link.STL
- added link right_hand_thumb_2_link, mass 0.02030626; collision mesh filename=package://g1_description/meshes/right_hand_thumb_2_link.STL; visual mesh filename=package://g1_description/meshes/right_hand_thumb_2_link.STL
- added link right_heel
- added link right_toe
- added link right_wrist_pitch_link, mass 0.48404956; collision mesh filename=package://g1_description/meshes/right_wrist_pitch_link.STL; visual mesh filename=package://g1_description/meshes/right_wrist_pitch_link.STL
- added link right_wrist_roll_link, mass 0.08544498; collision mesh filename=package://g1_description/meshes/right_wrist_roll_link.STL; visual mesh filename=package://g1_description/meshes/right_wrist_roll_link.STL
- added link right_wrist_yaw_link, mass 0.08457647; collision mesh filename=package://g1_description/meshes/right_wrist_yaw_link.STL; visual mesh filename=package://g1_description/meshes/right_wrist_yaw_link.STL
- added link waist_roll_link, mass 0.047; visual mesh filename=package://g1_description/meshes/waist_roll_link.STL
- added link waist_support_link, mass 0.001; collision mesh filename=package://g1_description/meshes/waist_support_link.STL; visual mesh filename=package://g1_description/meshes/waist_support_link.STL
- added link waist_yaw_link, mass 0.244; visual mesh filename=package://g1_description/meshes/waist_yaw_link.STL
- link head_link: mass 1.17976522 -> 1.036
- link left_ankle_roll_link: mass 0.391 -> 0.608; geometry collision sphere radius=0.005; collision sphere radius=0.005
- link left_hip_pitch_link: mass 1.299 -> 1.35
- link left_hip_roll_link: mass 1.446 -> 1.52
- link left_hip_yaw_link: mass 2.052 -> 1.702
- link left_knee_link: mass 2.252 -> 1.932; geometry collision mesh filename=package://g1_description/meshes/left_knee_link.STL; visual mesh filename=package://g1_description/meshes/left_knee_link.STL
- link left_shoulder_pitch_link: mass 0.713 -> 0.718; geometry collision cylinder length=0.05 radius=0.03; visual mesh filename=package://g1_description/meshes/left_shoulder_pitch_link.STL
- link left_shoulder_roll_link: mass 0.642 -> 0.643
- link left_shoulder_yaw_link: mass 0.713 -> 0.734
- link pelvis: mass 2.86 -> 3.813; geometry visual mesh filename=package://g1_description/meshes/pelvis.STL
- link pelvis_contour_link: mass None -> 0.001; geometry collision mesh filename=package://g1_description/meshes/pelvis_contour_link.STL; visual mesh filename=package://g1_description/meshes/pelvis_contour_link.STL
- link right_ankle_roll_link: mass 0.391 -> 0.608; geometry collision sphere radius=0.005; collision sphere radius=0.005
- link right_hip_pitch_link: mass 1.299 -> 1.35
- link right_hip_roll_link: mass 1.446 -> 1.52
- link right_hip_yaw_link: mass 2.052 -> 1.702
- link right_knee_link: mass 2.252 -> 1.932; geometry collision mesh filename=package://g1_description/meshes/right_knee_link.STL; visual mesh filename=package://g1_description/meshes/right_knee_link.STL
- link right_shoulder_pitch_link: mass 0.713 -> 0.718; geometry collision cylinder length=0.05 radius=0.03; visual mesh filename=package://g1_description/meshes/right_shoulder_pitch_link.S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
- link right_shoulder_roll_link: mass 0.642 -> 0.643
- link right_shoulder_yaw_link: mass 0.713 -> 0.734
- link torso_link: mass 6.33959811 -> 8.562
Joints:
- removed joint left_elbow_pitch_joint
- removed joint left_elbow_roll_joint
- removed joint left_five_joint
- removed joint left_four_joint
- removed joint left_one_joint
- removed joint left_palm_joint
- removed joint left_six_joint
- removed joint left_three_joint
- removed joint left_two_joint
- removed joint left_zero_joint
- removed joint right_elbow_pitch_joint
- removed joint right_elbow_roll_joint
- removed joint right_five_joint
- removed joint right_four_joint
- removed joint right_one_joint
- removed joint right_palm_joint
- removed joint right_six_joint
- removed joint right_three_joint
- removed joint right_two_joint
- removed joint right_zero_joint
- removed joint torso_joint
- added joint d435_joint: type fixed, parent torso_link, child d435_link, origin xyz=0.0576235 0.01753 0.41987 rpy=0 0.8307767239493009 0
- added joint left_elbow_joint: type revolute, parent left_shoulder_yaw_link, child left_elbow_link, origin xyz=0.015783 0 -0.080518 rpy=0 0 0, axis 0 1 0, limit lower=-1.0472 upper=2.0944 effort=25 velocity=12
- added joint left_hand_index_0_joint: type revolute, parent left_hand_palm_link, child left_hand_index_0_link, origin xyz=0.0777 0.0016 0.0285 rpy=0 0 0, axis 0 0 1, limit lower=-1.57079632 upper=0 effort=1.4 velocity=12
- added joint left_hand_index_1_joint: type revolute, parent left_hand_index_0_link, child left_hand_index_1_link, origin xyz=0.0458 0 0 rpy=0 0 0, axis 0 0 1, limit lower=-1.74532925 upper=0 effort=1.4 velocity=12
- added joint left_hand_middle_0_joint: type revolute, parent left_hand_palm_link, child left_hand_middle_0_link, origin xyz=0.0777 0.0016 -0.0285 rpy=0 0 0, axis 0 0 1, limit lower=-1.57079632 upper=0 effort=1.4 velocity=12
- added joint left_hand_middle_1_joint: type revolute, parent left_hand_middle_0_link, child left_hand_middle_1_link, origin xyz=0.0458 0 0 rpy=0 0 0, axis 0 0 1, limit lower=-1.74532925 upper=0 effort=1.4 velocity=12
- added joint left_hand_palm_joint: type fixed, parent left_wrist_yaw_link, child left_hand_palm_link, origin xyz=0.0415 0.003 0 rpy=0 0 0
- added joint left_hand_thumb_0_joint: type revolute, parent left_hand_palm_link, child left_hand_thumb_0_link, origin xyz=0.0255 0 0 rpy=0 0 0, axis 0 1 0, limit lower=-1.04719755 upper=1.04719755 effort=2.45 velocity=6.857
- added joint left_hand_thumb_1_joint: type revolute, parent left_hand_thumb_0_link, child left_hand_thumb_1_link, origin xyz=-0.0025 -0.0193 0 rpy=0 0 0, axis 0 0 1, limit lower=-0.72431163 upper=1.04719755 effort=1.4 velocity=12
- added joint left_hand_thumb_2_joint: type revolute, parent left_hand_thumb_1_link, child left_hand_thumb_2_link, origin xyz=0 -0.0458 0 rpy=0 0 0, axis 0 0 1, limit lower=0 upper=1.74532925 effort=1.4 velocity=12
- added joint left_heel_joint: type fixed, parent left_ankle_roll_link, child left_heel, origin xyz=-0.05 0 -0.03 rpy=0 0 0
- added joint left_toe_joint: type fixed, parent left_ankle_roll_link, child left_toe, origin xyz=0.12 0 -0.03 rpy=0 0 0
- added joint left_wrist_pitch_joint: type revolute, parent left_wrist_roll_link, child left_wrist_pitch_link, origin xyz=0.038 0 0 rpy=0 0 0, axis 0 1 0, limit lower=-1.614429558 upper=1.614429558 effort=5 velocity=22
- added joint left_wrist_roll_joint: type revolute, parent left_elbow_link, child left_wrist_roll_link, origin xyz=0.100 0.00188791 -0.010 rpy=0 0 0, axis 1 0 0, limit lower=-1.972222054 upper=1.972222054 effort=25 velocity=12
- added joint left_wrist_yaw_joint: type revolute, parent left_wrist_pitch_link, child left_wrist_yaw_link, origin xyz=0.046 0 0 rpy=0 0 0, axis 0 0 1, limit lower=-1.614429558 upper=1.614429558 effort=5 velocity=22
- added joint mid360_joint: type fixed, parent torso_link, child mid360_link, origin xyz=0.0002835 0.00003 0.40618 rpy=0 0.04014257279586953 0
- added joint right_elbow_joint: type revolute, parent right_shoulder_yaw_link, child right_elbow_link, origin xyz=0.015783 0 -0.080518 rpy=0 0 0, axis 0 1 0, limit lower=-1.0472 upper=2.0944 effort=25 velocity=12
- added joint right_hand_index_0_joint: type revolute, parent right_hand_palm_link, child right_hand_index_0_link, origin xyz=0.0777 -0.0016 0.0285 rpy=0 0 0, axis 0 0 1, limit lower=0 upper=1.57079632 effort=1.4 velocity=12
- added joint right_hand_index_1_joint: type revolute, parent right_hand_index_0_link, child right_hand_index_1_link, origin xyz=0.0458 0 0 rpy=0 0 0, axis 0 0 1, limit lower=0 upper=1.74532925 effort=1.4 velocity=12
- added joint right_hand_middle_0_joint: type revolute, parent right_hand_palm_link, child right_hand_middle_0_link, origin xyz=0.0777 -0.0016 -0.0285 rpy=0 0 0, axis 0 0 1, limit lower=0 upper=1.57079632 effort=1.4 velocity=12
- added joint right_hand_middle_1_joint: type revolute, parent right_hand_middle_0_link, child right_hand_middle_1_link, origin xyz=0.0458 0 0 rpy=0 0 0, axis 0 0 1, limit lower=0 upper=1.74532925 effort=1.4 velocity=12
- added joint right_hand_palm_joint: type fixed, parent right_wrist_yaw_link, child right_hand_palm_link, origin xyz=0.0415 -0.003 0 rpy=0 0 0
- added joint right_hand_thumb_0_joint: type revolute, parent right_hand_palm_link, child right_hand_thumb_0_link, origin xyz=0.0255 0 0 rpy=0 0 0, axis 0 1 0, limit lower=-1.04719755 upper=1.04719755 effort=2.45 velocity=6.857
- added joint right_hand_thumb_1_joint: type revolute, parent right_hand_thumb_0_link, child right_hand_thumb_1_link, origin xyz=-0.0025 0.0193 0 rpy=0 0 0, axis 0 0 1, limit lower=-1.04719755 upper=0.72431163 effort=1.4 velocity=12
- added joint right_hand_thumb_2_joint: type revolute, parent right_hand_thumb_1_link, child right_hand_thumb_2_link, origin xyz=0 0.0458 0 rpy=0 0 0, axis 0 0 1, limit lower=-1.74532925 upper=0 effort=1.4 velocity=12
- added joint right_heel_joint: type fixed, parent right_ankle_roll_link, child right_heel, origin xyz=-0.05 0 -0.03 rpy=0 0 0
- added joint right_toe_joint: type fixed, parent right_ankle_roll_link, child right_toe, origin xyz=0.12 0 -0.03 rpy=0 0 0
- added joint right_wrist_pitch_joint: type revolute, parent right_wrist_roll_link, child right_wrist_pitch_link, origin xyz=0.038 0 0 rpy=0 0 0, axis 0 1 0, limit lower=-1.614429558 upper=1.614429558 effort=5 velocity=22
- added joint right_wrist_roll_joint: type revolute, parent right_elbow_link, child right_wrist_roll_link, origin xyz=0.100 -0.00188791 -0.010 rpy=0 0 0, axis 1 0 0, limit lower=-1.972222054 upper=1.972222054 effort=25 velocity=12
- added joint right_wrist_yaw_joint: type revolute, parent right_wrist_pitch_link, child right_wrist_yaw_link, origin xyz=0.046 0 0 rpy=0 0 0, axis 0 0 1, limit lower=-1.614429558 upper=1.614429558 effort=5 velocity=22
- added joint waist_pitch_joint: type revolute, parent waist_roll_link, child torso_link, origin xyz=0 0 0.019 rpy=0 0 0, axis 0 1 0, limit lower=-0.52 upper=0.52 effort=50 velocity=12
- added joint waist_roll_joint: type revolute, parent waist_yaw_link, child waist_roll_link, origin xyz=-0.0039635 0 0.035 rpy=0 0 0, axis 1 0 0, limit lower=-0.52 upper=0.52 effort=50 velocity=12
- added joint waist_support_joint: type fixed, parent torso_link, child waist_support_link, origin xyz=0.0039635 0 -0.054 rpy=0 0 0
- added joint waist_yaw_joint: type revolute, parent pelvis, child waist_yaw_link, origin xyz=0 0 0 rpy=0 0 0, axis 0 0 1, limit lower=-2.618 upper=2.618 effort=88 velocity=12
- joint head_joint: origin xyz=0 0 0 rpy=0 0 0 -> xyz=0.0039635 0 -0.054 rpy=0 0 0
- joint imu_joint: origin xyz=-0.04233868314 0.00166 0.152067 rpy=0 0 0 -> xyz=-0.03959 -0.00224 0.13792 rpy=0 0 0
- joint left_ankle_pitch_joint: limit lower=-0.68 upper=0.73 effort=40 velocity=53 -> lower=-0.87267 upper=0.5236 effort=50 velocity=12; origin xyz=0 0.0040687 -0.30007 rpy=0 -0.16053 0 -> xyz=0 -9.4445E-05 -0.30001 rpy=0 0 0
- joint left_ankle_roll_joint: limit lower=-0.2618 upper=0.2618 effort=40 velocity=53 -> lower=-0.2618 upper=0.2618 effort=50 velocity=12
- joint left_hip_pitch_joint: limit lower=-2.35 upper=3.05 effort=88 velocity=32 -> lower=-2.5307 upper=2.8798 effort=88 velocity=12; origin xyz=0 0.06445 -0.1027 rpy=0 -0.34907 0 -> xyz=0 0.064452 -0.1027 rpy=0 0 0
- joint left_hip_roll_joint: limit lower=-0.26 upper=2.53 effort=88 velocity=32 -> lower=-0.5236 upper=2.9671 effort=88 velocity=12; origin xyz=0 0.0523 0 rpy=0 0 0 -> xyz=0 0.052 -0.030465 rpy=0 -0.1749 0
- joint left_hip_yaw_joint: limit lower=-2.75 upper=2.75 effort=88 velocity=32 -> lower=-2.7576 upper=2.7576 effort=88 velocity=12; origin xyz=0.01966 -0.0012139 -0.1241 rpy=0 0 0 -> xyz=0.025001 0 -0.12412 rpy=0 0 0
- joint left_knee_joint: limit lower=-0.33489 upper=2.5449 effort=139 velocity=20 -> lower=-0.087267 upper=2.8798 effort=139 velocity=12; origin xyz=-0.078292 -0.0017335 -0.177225 rpy=0 0.5096 0 -> xyz=-0.078273 0.0021489 -0.17734 rpy=0 0.1749 0
- joint left_shoulder_pitch_joint: limit lower=-2.9671 upper=2.7925 effort=21 velocity=53 -> lower=-3.0892 upper=2.6704 effort=25 velocity=12; origin xyz=-0.0025 0.10396 0.25928 rpy=0.27925 0 0 -> xyz=0.0039563 0.10022 0.23778 rpy=0.27931 5.4949E-05 -0.00019159
- joint left_shoulder_roll_joint: limit lower=-1.5882 upper=2.2515 effort=21 velocity=53 -> lower=-1.5882 upper=2.2515 effort=25 velocity=12; origin xyz=0 0.052 0 rpy=-0.27925 0 0 -> xyz=0 0.038 -0.013831 rpy=-0.27925 0 0
- joint left_shoulder_yaw_joint: limit lower=-2.618 upper=2.618 effort=21 velocity=53 -> lower=-2.618 upper=2.618 effort=25 velocity=12; origin xyz=-0.00354 0.0062424 -0.1032 rpy=0 0 0 -> xyz=0 0.00624 -0.1032 rpy=0 0 0
- joint logo_joint: origin xyz=0 0 0 rpy=0 0 0 -> xyz=0.0039635 0 -0.054 rpy=0 0 0
- joint right_ankle_pitch_joint: limit lower=-0.68 upper=0.73 effort=40 velocity=53 -> lower=-0.87267 upper=0.5236 effort=50 velocity=12; origin xyz=0 -0.0040687 -0.30007 rpy=0 -0.16053 0 -> xyz=0 9.4445E-05 -0.30001 rpy=0 0 0
- joint right_ankle_roll_joint: limit lower=-0.2618 upper=0.2618 effort=40 velocity=53 -> lower=-0.2618 upper=0.2618 effort=50 velocity=12
- joint right_hip_pitch_joint: limit lower=-2.35 upper=3.05 effort=88 velocity=32 -> lower=-2.5307 upper=2.8798 effort=88 velocity=12; origin xyz=0 -0.06445 -0.1027 rpy=0 -0.34907 0 -> xyz=0 -0.064452 -0.1027 rpy=0 0 0
- joint right_hip_roll_joint: limit lower=-2.53 upper=0.26 effort=88 velocity=32 -> lower=-2.9671 upper=0.5236 effort=88 velocity=12; origin xyz=0 -0.0523 0 rpy=0 0 0 -> xyz=0 -0.052 -0.030465 rpy=0 -0.1749 0
- joint right_hip_yaw_joint: limit lower=-2.75 upper=2.75 effort=88 velocity=32 -> lower=-2.7576 upper=2.7576 effort=88 velocity=12; origin xyz=0.01966 0.0012139 -0.1241 rpy=0 0 0 -> xyz=0.025001 0 -0.12412 rpy=0 0 0
- joint right_knee_joint: limit lower=-0.33489 upper=2.5449 effort=139 velocity=20 -> lower=-0.087267 upper=2.8798 effort=139 velocity=12; origin xyz=-0.078292 0.0017335 -0.177225 rpy=0 0.5096 0 -> xyz=-0.078273 -0.0021489 -0.17734 rpy=0 0.1749 0
- joint right_shoulder_pitch_joint: limit lower=-2.9671 upper=2.7925 effort=21 velocity=53 -> lower=-3.0892 upper=2.6704 effort=25 velocity=12; origin xyz=-0.0025 -0.10396 0.25928 rpy=-0.27925 0 0 -> xyz=0.0039563 -0.10021 0.23778 rpy=-0.27931 5.4949E-05 0.00019159
- joint right_shoulder_roll_joint: limit lower=-2.2515 upper=1.5882 effort=21 velocity=53 -> lower=-2.2515 upper=1.5882 effort=25 velocity=12; origin xyz=0 -0.052 0 rpy=0.27925 0 0 -> xyz=0 -0.038 -0.013831 rpy=0.27925 0 0
- joint right_shoulder_yaw_joint: limit lower=-2.618 upper=2.618 effort=21 velocity=53 -> lower=-2.618 upper=2.618 effort=25 velocity=12; origin xyz=-0.00354 -0.0062424 -0.1032 rpy=0 0 0 -> xyz=0 -0.00624 -0.1032 rpy=0 0 0
