Commit message: worked on setting up foxglove visualization

File: obelisk_ws/src/robots/d1_description/urdf/d1.urdf (robot description, URDF)
Before this commit: robot d1_description, 9 links, 8 joints
Joints:
- removed joint Joint1
- removed joint Joint2
- removed joint Joint3
- removed joint Joint4
- removed joint Joint5
- removed joint Joint6
- removed joint Joint7_1
- removed joint Joint7_2
- added joint angle0: type revolute, parent base_link, child Link1, origin xyz=0 0 0.0533 rpy=0 0 -3.1416, axis 0 0 1, limit lower=-2.35 upper=2.35 effort=0 velocity=0
- added joint angle1: type revolute, parent Link1, child Link2, origin xyz=0 0.028 0.0563 rpy=1.5708 0 -3.1416, axis 0 0 -1, limit lower=-1.57 upper=1.57 effort=0 velocity=0
- added joint angle2: type revolute, parent Link2, child Link3, origin xyz=0 0.2693 0.0009 rpy=0 0 0, axis 0 0 -1, limit lower=-1.57 upper=1.57 effort=0 velocity=0
- added joint angle3: type revolute, parent Link3, child Link4, origin xyz=0.0577 0.042 -0.0275 rpy=-1.5708 0 -1.5708, axis 0 0 1, limit lower=-2.35 upper=2.35 effort=0 velocity=0
- added joint angle4: type revolute, parent Link4, child Link5, origin xyz=-0.0001 -0.0237 0.14018 rpy=1.5708 -1.5708 0, axis 0 0 -1, limit lower=-1.57 upper=1.57 effort=0 velocity=0
- added joint angle5: type revolute, parent Link5, child Link6, origin xyz=0.0825 -0.0010782 -0.023822 rpy=-1.5708 0 -1.5708, axis 0 0 -1, limit lower=-2.35 upper=2.35 effort=0 velocity=0
- added joint angle6: type prismatic, parent Link6, child Link7_1, origin xyz=-0.0056012 -0.029636 0.0706 rpy=-1.5714 -1.5708 0, axis 0 0 -1, limit lower=0 upper=0.03 effort=0 velocity=0
- added joint angle6_2: type prismatic, parent Link6, child Link7_2, origin xyz=-0.0056388 0.02964 0.0706 rpy=1.5702 -1.5708 0, axis 0 0 1, limit lower=-0.03 upper=0 effort=0 velocity=0

Commit message: fixed control input to joint6

File: obelisk_ws/src/robots/d1_description/urdf/d1.urdf (robot description, URDF)
Before this commit: robot d1_description, 9 links, 8 joints
Joints:
- removed joint angle0
- removed joint angle1
- removed joint angle2
- removed joint angle3
- removed joint angle4
- removed joint angle5
- removed joint angle6
- removed joint angle6_2
- added joint joint0: type revolute, parent base_link, child Link1, origin xyz=0 0 0.0533 rpy=0 0 -3.1416, axis 0 0 1, limit lower=-2.35 upper=2.35 effort=0 velocity=0
- added joint joint1: type revolute, parent Link1, child Link2, origin xyz=0 0.028 0.0563 rpy=1.5708 0 -3.1416, axis 0 0 -1, limit lower=-1.57 upper=1.57 effort=0 velocity=0
- added joint joint2: type revolute, parent Link2, child Link3, origin xyz=0 0.2693 0.0009 rpy=0 0 0, axis 0 0 -1, limit lower=-1.57 upper=1.57 effort=0 velocity=0
- added joint joint3: type revolute, parent Link3, child Link4, origin xyz=0.0577 0.042 -0.0275 rpy=-1.5708 0 -1.5708, axis 0 0 1, limit lower=-2.35 upper=2.35 effort=0 velocity=0
- added joint joint4: type revolute, parent Link4, child Link5, origin xyz=-0.0001 -0.0237 0.14018 rpy=1.5708 -1.5708 0, axis 0 0 -1, limit lower=-1.57 upper=1.57 effort=0 velocity=0
- added joint joint5: type revolute, parent Link5, child Link6, origin xyz=0.0825 -0.0010782 -0.023822 rpy=-1.5708 0 -1.5708, axis 0 0 -1, limit lower=-2.35 upper=2.35 effort=0 velocity=0
- added joint joint6: type prismatic, parent Link6, child Link7_1, origin xyz=-0.0056012 -0.029636 0.0706 rpy=-1.5714 -1.5708 0, axis 0 0 -1, limit lower=0 upper=0.03 effort=0 velocity=0
- added joint joint6_2: type prismatic, parent Link6, child Link7_2, origin xyz=-0.0056388 0.02964 0.0706 rpy=1.5702 -1.5708 0, axis 0 0 1, limit lower=-0.03 upper=0 effort=0 velocity=0

Commit message: fixed gripper control code, set control limits, cleaned code

File: obelisk_ws/src/robots/d1_description/urdf/d1.urdf (robot description, URDF)
Before this commit: robot d1_description, 9 links, 8 joints
Joints:
- removed joint joint0
- removed joint joint6_2
- added joint gripper1: type prismatic, parent Link6, child Link7_1, origin xyz=-0.0056012 -0.029636 0.0706 rpy=-1.5714 -1.5708 0, axis 0 0 -1, limit lower=0 upper=0.03 effort=0 velocity=0
- added joint gripper2: type prismatic, parent Link6, child Link7_2, origin xyz=-0.0056388 0.02964 0.0706 rpy=1.5702 -1.5708 0, axis 0 0 1, limit lower=-0.03 upper=0 effort=0 velocity=0
- joint joint1: axis 0 0 -1 -> 0 0 1; child Link2 -> Link1; limit lower=-1.57 upper=1.57 effort=0 velocity=0 -> lower=-2.35 upper=2.35 effort=0 velocity=0; origin xyz=0 0.028 0.0563 rpy=1.5708 0 -3.1416 -> xyz=0 0 0.0533 rpy=0 0 -3.1416; parent Link1 -> base_link
- joint joint2: child Link3 -> Link2; origin xyz=0 0.2693 0.0009 rpy=0 0 0 -> xyz=0 0.028 0.0563 rpy=1.5708 0 -3.1416; parent Link2 -> Link1
- joint joint3: axis 0 0 1 -> 0 0 -1; child Link4 -> Link3; limit lower=-2.35 upper=2.35 effort=0 velocity=0 -> lower=-1.57 upper=1.57 effort=0 velocity=0; origin xyz=0.0577 0.042 -0.0275 rpy=-1.5708 0 -1.5708 -> xyz=0 0.2693 0.0009 rpy=0 0 0; parent Link3 -> Link2
- joint joint4: axis 0 0 -1 -> 0 0 1; child Link5 -> Link4; limit lower=-1.57 upper=1.57 effort=0 velocity=0 -> lower=-2.35 upper=2.35 effort=0 velocity=0; origin xyz=-0.0001 -0.0237 0.14018 rpy=1.5708 -1.5708 0 -> xyz=0.0577 0.042 -0.0275 rpy=-1.5708 0 -1.5708; parent Link4 -> Link3
- joint joint5: child Link6 -> Link5; limit lower=-2.35 upper=2.35 effort=0 velocity=0 -> lower=-1.57 upper=1.57 effort=0 velocity=0; origin xyz=0.0825 -0.0010782 -0.023822 rpy=-1.5708 0 -1.5708 -> xyz=-0.0001 -0.0237 0.14018 rpy=1.5708 -1.5708 0; parent Link5 -> Link4
- joint joint6: child Link7_1 -> Link6; limit lower=0 upper=0.03 effort=0 velocity=0 -> lower=-2.35 upper=2.35 effort=0 velocity=0; origin xyz=-0.0056012 -0.029636 0.0706 rpy=-1.5714 -1.5708 0 -> xyz=0.0825 -0.0010782 -0.023822 rpy=-1.5708 0 -1.5708; parent Link6 -> Link5; type prismatic -> revolute

Commit message: increase precision

File: obelisk_ws/src/robots/d1_description/urdf/d1.urdf (robot description, URDF)
Before this commit: robot d1_description, 9 links, 8 joints
Joints:
- joint gripper1: origin xyz=-0.0056012 -0.029636 0.0706 rpy=-1.5714 -1.5708 0 -> xyz=-0.0056012 -0.029636 0.0706 rpy=-1.57079632679 -1.57079632679 0
- joint gripper2: origin xyz=-0.0056388 0.02964 0.0706 rpy=1.5702 -1.5708 0 -> xyz=-0.0056388 0.02964 0.0706 rpy=1.57079632679 -1.57079632679 0
- joint joint1: origin xyz=0 0 0.0533 rpy=0 0 -3.1416 -> xyz=0 0 0.0533 rpy=0 0 -3.14159265358
- joint joint2: limit lower=-1.57 upper=1.57 effort=0 velocity=0 -> lower=-1.57079632679 upper=1.57079632679 effort=0 velocity=0; origin xyz=0 0.028 0.0563 rpy=1.5708 0 -3.1416 -> xyz=0 0.028 0.0563 rpy=1.57079632679 0 -3.14159265358
- joint joint3: limit lower=-1.57 upper=1.57 effort=0 velocity=0 -> lower=-1.57079632679 upper=1.57079632679 effort=0 velocity=0
- joint joint4: origin xyz=0.0577 0.042 -0.0275 rpy=-1.5708 0 -1.5708 -> xyz=0.0577 0.042 -0.0275 rpy=-1.57079632679 0 -1.57079632679
- joint joint5: limit lower=-1.57 upper=1.57 effort=0 velocity=0 -> lower=-1.57079632679 upper=1.57079632679 effort=0 velocity=0; origin xyz=-0.0001 -0.0237 0.14018 rpy=1.5708 -1.5708 0 -> xyz=-0.0001 -0.0237 0.14018 rpy=1.57079632679 -1.57079632679 0
- joint joint6: origin xyz=0.0825 -0.0010782 -0.023822 rpy=-1.5708 0 -1.5708 -> xyz=0.0825 -0.0010782 -0.023822 rpy=-1.57079632679 0 -1.57079632679

Commit message: edit urdf revolute joint axis

File: obelisk_ws/src/robots/d1_description/urdf/d1.urdf (robot description, URDF)
Before this commit: robot d1_description, 9 links, 8 joints
Joints:
- joint joint3: axis 0 0 1 -> 0 0 -1
- joint joint4: axis 0 0 1 -> 0 0 -1
