Commit message: urdf to match xml and depth scan

File: obelisk_ws/src/robots/themis_description/urdf/themis.urdf (robot description, URDF)
Before this commit: robot TH02-A7, 29 links, 28 joints
Links:
- link ANKLE_L: mass 0.01 -> 0.006946; geometry collision mesh filename=../meshes/ANKLE_L.STL; visual mesh filename=../meshes/ANKLE_L.STL
- link ANKLE_R: mass 0.01 -> 0.006946; geometry collision mesh filename=../meshes/ANKLE_R.STL; visual mesh filename=../meshes/ANKLE_R.STL
- link BASE_LINK: mass 12.72953 -> 12.72; geometry collision mesh filename=../meshes/BASE_LINK.STL; visual mesh filename=../meshes/BASE_LINK.STL
- link ELBOW_L: mass 0.37854 -> 0.37853; geometry collision mesh filename=../meshes/ELBOW_L.STL; visual mesh filename=../meshes/ELBOW_L.STL
- link ELBOW_R: geometry collision mesh filename=../meshes/ELBOW_R.STL; visual mesh filename=../meshes/ELBOW_R.STL
- link FEMUR_L: mass 3.75393 -> 3.75384; geometry collision mesh filename=../meshes/FEMUR_L.STL; visual mesh filename=../meshes/FEMUR_L.STL
- link FEMUR_R: geometry collision mesh filename=../meshes/FEMUR_R.STL; visual mesh filename=../meshes/FEMUR_R.STL
- link FOOT_L: geometry collision box size=0.01 0.1 0.235; visual mesh filename=../meshes/FOOT_L.STL
- link FOOT_R: geometry collision box size=0.01 0.1 0.235; visual mesh filename=../meshes/FOOT_R.STL
- link FOREARM_L: geometry collision mesh filename=../meshes/FOREARM_L.STL; visual mesh filename=../meshes/FOREARM_L.STL
- link FOREARM_R: geometry collision mesh filename=../meshes/FOREARM_R.STL; visual mesh filename=../meshes/FOREARM_R.STL
- link HEAD: geometry collision mesh filename=../meshes/HEAD.STL; visual mesh filename=../meshes/HEAD.STL
- link HIP_ABAD_L: mass 2.818 -> 2.78794; geometry collision mesh filename=../meshes/HIP_ABAD_L.STL; visual mesh filename=../meshes/HIP_ABAD_L.STL
- link HIP_ABAD_R: geometry collision mesh filename=../meshes/HIP_ABAD_R.STL; visual mesh filename=../meshes/HIP_ABAD_R.STL
- link HIP_L: geometry collision mesh filename=../meshes/HIP_L.STL; visual mesh filename=../meshes/HIP_L.STL
- link HIP_R: geometry collision mesh filename=../meshes/HIP_R.STL; visual mesh filename=../meshes/HIP_R.STL
- link LOWERSHOULDER_L: geometry collision mesh filename=../meshes/LOWERSHOULDER_L.STL; visual mesh filename=../meshes/LOWERSHOULDER_L.STL
- link LOWERSHOULDER_R: geometry collision mesh filename=../meshes/LOWERSHOULDER_R.STL; visual mesh filename=../meshes/LOWERSHOULDER_R.STL
- link LOWERWRIST_L: geometry collision sphere radius=0.04; visual mesh filename=../meshes/LOWERWRIST_L.STL
- link LOWERWRIST_R: geometry collision sphere radius=0.04; visual mesh filename=../meshes/LOWERWRIST_R.STL
- link NECK: geometry collision mesh filename=../meshes/NECK.STL; visual mesh filename=../meshes/NECK.STL
- link TIBIA_L: geometry collision mesh filename=../meshes/TIBIA_L.STL; visual mesh filename=../meshes/TIBIA_L.STL
- link TIBIA_R: geometry collision mesh filename=../meshes/TIBIA_R.STL; visual mesh filename=../meshes/TIBIA_R.STL
- link UPPERARM_L: geometry collision mesh filename=../meshes/UPPERARM_L.STL; visual mesh filename=../meshes/UPPERARM_L.STL
- link UPPERARM_R: geometry collision mesh filename=../meshes/UPPERARM_R.STL; visual mesh filename=../meshes/UPPERARM_R.STL
- link UPPERSHOULDER_L: geometry collision mesh filename=../meshes/UPPERSHOULDER_L.STL; visual mesh filename=../meshes/UPPERSHOULDER_L.STL
- link UPPERSHOULDER_R: geometry collision mesh filename=../meshes/UPPERSHOULDER_R.STL; visual mesh filename=../meshes/UPPERSHOULDER_R.STL
- link UPPERWRIST_L: geometry collision mesh filename=../meshes/UPPERWRIST_L.STL; visual mesh filename=../meshes/UPPERWRIST_L.STL
- link UPPERWRIST_R: geometry collision mesh filename=../meshes/UPPERWRIST_R.STL; visual mesh filename=../meshes/UPPERWRIST_R.STL
